Commit message: Update g1_23dof.urdf

File: robots/g1_description/g1_23dof.urdf (robot description, URDF)
Before this commit: robot g1_23dof, 33 links, 32 joints
Links:
- link head_link: geometry collision mesh filename=package://g1_description/head_link.STL; visual mesh filename=package://g1_description/head_link.STL
- link left_ankle_pitch_link: geometry collision mesh filename=package://g1_description/left_ankle_pitch_link.STL; visual mesh filename=package://g1_description/left_ankle_pitch_link.STL
- link left_ankle_roll_link: geometry collision sphere radius=0.005; collision sphere radius=0.005
- link left_elbow_link: geometry collision mesh filename=package://g1_description/left_elbow_link.STL; visual mesh filename=package://g1_description/left_elbow_link.STL
- link left_hip_pitch_link: geometry collision mesh filename=package://g1_description/left_hip_pitch_link.STL; visual mesh filename=package://g1_description/left_hip_pitch_link.STL
- link left_hip_roll_link: geometry collision mesh filename=package://g1_description/left_hip_roll_link.STL; visual mesh filename=package://g1_description/left_hip_roll_link.STL
- link left_hip_yaw_link: geometry collision mesh filename=package://g1_description/left_hip_yaw_link.STL; visual mesh filename=package://g1_description/left_hip_yaw_link.STL
- link left_knee_link: geometry collision mesh filename=package://g1_description/left_knee_link.STL; visual mesh filename=package://g1_description/left_knee_link.STL
- link left_shoulder_pitch_link: geometry collision cylinder length=0.05 radius=0.03; visual mesh filename=package://g1_description/left_shoulder_pitch_link.STL
- link left_shoulder_roll_link: geometry collision cylinder length=0.03 radius=0.03; visual mesh filename=package://g1_description/left_shoulder_roll_link.STL
- link left_shoulder_yaw_link: geometry collision mesh filename=package://g1_description/left_shoulder_yaw_link.STL; visual mesh filename=package://g1_description/left_shoulder_yaw_link.STL
- link left_wrist_roll_rubber_hand: geometry collision mesh filename=package://g1_description/left_wrist_roll_rubber_hand.STL; visual mesh filename=package://g1_description/left_wrist_roll_rubber_hand.STL
- link logo_link: geometry collision mesh filename=package://g1_description/logo_link.STL; visual mesh filename=package://g1_description/logo_link.STL
- link pelvis: geometry visual mesh filename=package://g1_description/pelvis.STL
- link pelvis_contour_link: geometry collision mesh filename=package://g1_description/pelvis_contour_link.STL; visual mesh filename=package://g1_description/pelvis_contour_link.STL
- link right_ankle_pitch_link: geometry collision mesh filename=package://g1_description/right_ankle_pitch_link.STL; visual mesh filename=package://g1_description/right_ankle_pitch_link.STL
- link right_ankle_roll_link: geometry collision sphere radius=0.005; collision sphere radius=0.005
- link right_elbow_link: geometry collision mesh filename=package://g1_description/right_elbow_link.STL; visual mesh filename=package://g1_description/right_elbow_link.STL
- link right_hip_pitch_link: geometry collision mesh filename=package://g1_description/right_hip_pitch_link.STL; visual mesh filename=package://g1_description/right_hip_pitch_link.STL
- link right_hip_roll_link: geometry collision mesh filename=package://g1_description/right_hip_roll_link.STL; visual mesh filename=package://g1_description/right_hip_roll_link.STL
- link right_hip_yaw_link: geometry collision mesh filename=package://g1_description/right_hip_yaw_link.STL; visual mesh filename=package://g1_description/right_hip_yaw_link.STL
- link right_knee_link: geometry collision mesh filename=package://g1_description/right_knee_link.STL; visual mesh filename=package://g1_description/right_knee_link.STL
- link right_shoulder_pitch_link: geometry collision cylinder length=0.05 radius=0.03; visual mesh filename=package://g1_description/right_shoulder_pitch_link.STL
- link right_shoulder_roll_link: geometry collision cylinder length=0.03 radius=0.03; visual mesh filename=package://g1_description/right_shoulder_roll_link.STL
- link right_shoulder_yaw_link: geometry collision mesh filename=package://g1_description/right_shoulder_yaw_link.STL; visual mesh filename=package://g1_description/right_shoulder_yaw_link.STL
- link right_wrist_roll_rubber_hand: geometry collision mesh filename=package://g1_description/right_wrist_roll_rubber_hand.STL; visual mesh filename=package://g1_description/right_wrist_roll_rubber_hand.STL
- link torso_link: geometry collision mesh filename=package://g1_description/torso_link.STL; visual mesh filename=package://g1_description/torso_link.STL
- link waist_support_link: geometry collision mesh filename=package://g1_description/waist_support_link.STL; visual mesh filename=package://g1_description/waist_support_link.STL
- link waist_yaw_fixed_link: geometry visual mesh filename=package://g1_description/waist_yaw_link.STL

Commit message: Update g1_23dof.urdf

File: robots/g1_description/g1_23dof.urdf (robot description, URDF)
Before this commit: robot g1_23dof, 33 links, 32 joints
Links:
- link head_link: geometry collision mesh filename=package://g1_description/meshes/head_link.STL; visual mesh filename=package://g1_description/meshes/head_link.STL
- link left_ankle_pitch_link: geometry collision mesh filename=package://g1_description/meshes/left_ankle_pitch_link.STL; visual mesh filename=package://g1_description/meshes/left_ankle_pitch_link.STL
- link left_ankle_roll_link: geometry collision sphere radius=0.005; collision sphere radius=0.005
- link left_elbow_link: geometry collision mesh filename=package://g1_description/meshes/left_elbow_link.STL; visual mesh filename=package://g1_description/meshes/left_elbow_link.STL
- link left_hip_pitch_link: geometry collision mesh filename=package://g1_description/meshes/left_hip_pitch_link.STL; visual mesh filename=package://g1_description/meshes/left_hip_pitch_link.STL
- link left_hip_roll_link: geometry collision mesh filename=package://g1_description/meshes/left_hip_roll_link.STL; visual mesh filename=package://g1_description/meshes/left_hip_roll_link.STL
- link left_hip_yaw_link: geometry collision mesh filename=package://g1_description/meshes/left_hip_yaw_link.STL; visual mesh filename=package://g1_description/meshes/left_hip_yaw_link.STL
- link left_knee_link: geometry collision mesh filename=package://g1_description/meshes/left_knee_link.STL; visual mesh filename=package://g1_description/meshes/left_knee_link.STL
- link left_shoulder_pitch_link: geometry collision cylinder length=0.05 radius=0.03; visual mesh filename=package://g1_description/meshes/left_shoulder_pitch_link.STL
- link left_shoulder_roll_link: geometry collision cylinder length=0.03 radius=0.03; visual mesh filename=package://g1_description/meshes/left_shoulder_roll_link.STL
- link left_shoulder_yaw_link: geometry collision mesh filename=package://g1_description/meshes/left_shoulder_yaw_link.STL; visual mesh filename=package://g1_description/meshes/left_shoulder_yaw_link.STL
- link left_wrist_roll_rubber_hand: geometry collision mesh filename=package://g1_description/meshes/left_wrist_roll_rubber_hand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; visual mesh filename=package://g1_description/meshes/left_wrist_roll_rubber_hand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
- link logo_link: geometry collision mesh filename=package://g1_description/meshes/logo_link.STL; visual mesh filename=package://g1_description/meshes/logo_link.STL
- link pelvis: geometry visual mesh filename=package://g1_description/meshes/pelvis.STL
- link pelvis_contour_link: geometry collision mesh filename=package://g1_description/meshes/pelvis_contour_link.STL; visual mesh filename=package://g1_description/meshes/pelvis_contour_link.STL
- link right_ankle_pitch_link: geometry collision mesh filename=package://g1_description/meshes/right_ankle_pitch_link.STL; visual mesh filename=package://g1_description/meshes/right_ankle_pitch_link.STL
- link right_ankle_roll_link: geometry collision sphere radius=0.005; collision sphere radius=0.005
- link right_elbow_link: geometry collision mesh filename=package://g1_description/meshes/right_elbow_link.STL; visual mesh filename=package://g1_description/meshes/right_elbow_link.STL
- link right_hip_pitch_link: geometry collision mesh filename=package://g1_description/meshes/right_hip_pitch_link.STL; visual mesh filename=package://g1_description/meshes/right_hip_pitch_link.STL
- link right_hip_roll_link: geometry collision mesh filename=package://g1_description/meshes/right_hip_roll_link.STL; visual mesh filename=package://g1_description/meshes/right_hip_roll_link.STL
- link right_hip_yaw_link: geometry collision mesh filename=package://g1_description/meshes/right_hip_yaw_link.STL; visual mesh filename=package://g1_description/meshes/right_hip_yaw_link.STL
- link right_knee_link: geometry collision mesh filename=package://g1_description/meshes/right_knee_link.STL; visual mesh filename=package://g1_description/meshes/right_knee_link.STL
- link right_shoulder_pitch_link: geometry collision cylinder length=0.05 radius=0.03; visual mesh filename=package://g1_description/meshes/right_shoulder_pitch_link.S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
- link right_shoulder_roll_link: geometry collision cylinder length=0.03 radius=0.03; visual mesh filename=package://g1_description/meshes/right_shoulder_roll_link.STL
- link right_shoulder_yaw_link: geometry collision mesh filename=package://g1_description/meshes/right_shoulder_yaw_link.STL; visual mesh filename=package://g1_description/meshes/right_shoulder_yaw_link.STL
- link right_wrist_roll_rubber_hand: geometry collision mesh filename=package://g1_description/meshes/right_wrist_roll_rubber_han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; visual mesh filename=package://g1_description/meshes/right_wrist_roll_rubber_han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
- link torso_link: geometry collision mesh filename=package://g1_description/meshes/torso_link.STL; visual mesh filename=package://g1_description/meshes/torso_link.STL
- link waist_support_link: geometry collision mesh filename=package://g1_description/meshes/waist_support_link.STL; visual mesh filename=package://g1_description/meshes/waist_support_link.STL
- link waist_yaw_fixed_link: geometry visual mesh filename=package://g1_description/meshes/waist_yaw_link.STL
