Commit message: Update g1_29dof_rev_1_0_with_inspire_hand_FTP.urdf

File: robots/g1_description/g1_29dof_rev_1_0_with_inspire_hand_FTP.urdf (robot description, URDF)
Before this commit: robot g1_29dof_rev_1_0_with_inspire_hand_FTP, 97 links, 96 joints
Links:
- link head_link: geometry collision mesh filename=package://g1_description/meshes/head_link.STL; visual mesh filename=package://g1_description/meshes/head_link.STL
- link left_ankle_pitch_link: geometry collision mesh filename=package://g1_description/meshes/left_ankle_pitch_link.STL; visual mesh filename=package://g1_description/meshes/left_ankle_pitch_link.STL
- link left_ankle_roll_link: geometry collision sphere radius=0.005; collision sphere radius=0.005
- link left_base_link: geometry collision mesh filename=package://g1_description/meshes/left_base_link.STL; visual mesh filename=package://g1_description/meshes/left_base_link.STL
- link left_elbow_link: geometry collision mesh filename=package://g1_description/meshes/left_elbow_link.STL; visual mesh filename=package://g1_description/meshes/left_elbow_link.STL
- link left_hip_pitch_link: geometry collision mesh filename=package://g1_description/meshes/left_hip_pitch_link.STL; visual mesh filename=package://g1_description/meshes/left_hip_pitch_link.STL
- link left_hip_roll_link: geometry collision mesh filename=package://g1_description/meshes/left_hip_roll_link.STL; visual mesh filename=package://g1_description/meshes/left_hip_roll_link.STL
- link left_hip_yaw_link: geometry collision mesh filename=package://g1_description/meshes/left_hip_yaw_link.STL; visual mesh filename=package://g1_description/meshes/left_hip_yaw_link.STL
- link left_index_1: geometry collision mesh filename=package://g1_description/meshes/left_index_1.STL; visual mesh filename=package://g1_description/meshes/left_index_1.STL
- link left_index_2: geometry collision mesh filename=package://g1_description/meshes/left_index_2.STL; visual mesh filename=package://g1_description/meshes/left_index_2.STL
- link left_index_force_sensor_1: geometry collision mesh filename=package://g1_description/meshes/left_index_force_sensor_1.S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; visual mesh filename=package://g1_description/meshes/left_index_force_sensor_1.S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
- link left_index_force_sensor_2: geometry collision mesh filename=package://g1_description/meshes/left_index_force_sensor_2.S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; visual mesh filename=package://g1_description/meshes/left_index_force_sensor_2.S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
- link left_index_force_sensor_3: geometry collision mesh filename=package://g1_description/meshes/left_index_force_sensor_3.S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; visual mesh filename=package://g1_description/meshes/left_index_force_sensor_3.S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
- link left_knee_link: geometry collision mesh filename=package://g1_description/meshes/left_knee_link.STL; visual mesh filename=package://g1_description/meshes/left_knee_link.STL
- link left_little_1: geometry collision mesh filename=package://g1_description/meshes/left_little_1.STL; visual mesh filename=package://g1_description/meshes/left_little_1.STL
- link left_little_2: geometry collision mesh filename=package://g1_description/meshes/left_little_2.STL; visual mesh filename=package://g1_description/meshes/left_little_2.STL
- link left_little_force_sensor_1: geometry collision mesh filename=package://g1_description/meshes/left_little_force_sensor_1.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; visual mesh filename=package://g1_description/meshes/left_little_force_sensor_1.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
- link left_little_force_sensor_2: geometry collision mesh filename=package://g1_description/meshes/left_little_force_sensor_2.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; visual mesh filename=package://g1_description/meshes/left_little_force_sensor_2.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
- link left_little_force_sensor_3: geometry collision mesh filename=package://g1_description/meshes/left_little_force_sensor_3.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; visual mesh filename=package://g1_description/meshes/left_little_force_sensor_3.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
- link left_middle_1: geometry collision mesh filename=package://g1_description/meshes/left_middle_1.STL; visual mesh filename=package://g1_description/meshes/left_middle_1.STL
- link left_middle_2: geometry collision mesh filename=package://g1_description/meshes/left_middle_2.STL; visual mesh filename=package://g1_description/meshes/left_middle_2.STL
- link left_middle_force_sensor_1: geometry collision mesh filename=package://g1_description/meshes/left_middle_force_sensor_1.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; visual mesh filename=package://g1_description/meshes/left_middle_force_sensor_1.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
- link left_middle_force_sensor_2: geometry collision mesh filename=package://g1_description/meshes/left_middle_force_sensor_2.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; visual mesh filename=package://g1_description/meshes/left_middle_force_sensor_2.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
- link left_middle_force_sensor_3: geometry collision mesh filename=package://g1_description/meshes/left_middle_force_sensor_3.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; visual mesh filename=package://g1_description/meshes/left_middle_force_sensor_3.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
- link left_palm_force_sensor: geometry collision mesh filename=package://g1_description/meshes/left_palm_force_sensor.STL; visual mesh filename=package://g1_description/meshes/left_palm_force_sensor.STL
- link left_ring_1: geometry collision mesh filename=package://g1_description/meshes/left_ring_1.STL; visual mesh filename=package://g1_description/meshes/left_ring_1.STL
- link left_ring_2: geometry collision mesh filename=package://g1_description/meshes/left_ring_2.STL; visual mesh filename=package://g1_description/meshes/left_ring_2.STL
- link left_ring_force_sensor_1: geometry collision mesh filename=package://g1_description/meshes/left_ring_force_sensor_1.STL; visual mesh filename=package://g1_description/meshes/left_ring_force_sensor_1.STL
- link left_ring_force_sensor_2: geometry collision mesh filename=package://g1_description/meshes/left_ring_force_sensor_2.STL; visual mesh filename=package://g1_description/meshes/left_ring_force_sensor_2.STL
- link left_ring_force_sensor_3: geometry collision mesh filename=package://g1_description/meshes/left_ring_force_sensor_3.STL; visual mesh filename=package://g1_description/meshes/left_ring_force_sensor_3.STL
- link left_shoulder_pitch_link: geometry collision cylinder length=0.05 radius=0.03; visual mesh filename=package://g1_description/meshes/left_shoulder_pitch_link.STL
- link left_shoulder_roll_link: geometry collision cylinder length=0.03 radius=0.03; visual mesh filename=package://g1_description/meshes/left_shoulder_roll_link.STL
- link left_shoulder_yaw_link: geometry collision mesh filename=package://g1_description/meshes/left_shoulder_yaw_link.STL; visual mesh filename=package://g1_description/meshes/left_shoulder_yaw_link.STL
- link left_thumb_1: geometry collision mesh filename=package://g1_description/meshes/left_thumb_1.STL; visual mesh filename=package://g1_description/meshes/left_thumb_1.STL
- link left_thumb_2: geometry collision mesh filename=package://g1_description/meshes/left_thumb_2.STL; visual mesh filename=package://g1_description/meshes/left_thumb_2.STL
- link left_thumb_3: geometry collision mesh filename=package://g1_description/meshes/left_thumb_3.STL; visual mesh filename=package://g1_description/meshes/left_thumb_3.STL
- link left_thumb_4: geometry collision mesh filename=package://g1_description/meshes/left_thumb_4.STL; visual mesh filename=package://g1_description/meshes/left_thumb_4.STL
- link left_thumb_force_sensor_1: geometry collision mesh filename=package://g1_description/meshes/left_thumb_force_sensor_1.S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; visual mesh filename=package://g1_description/meshes/left_thumb_force_sensor_1.S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
- link left_thumb_force_sensor_2: geometry collision mesh filename=package://g1_description/meshes/left_thumb_force_sensor_2.S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; visual mesh filename=package://g1_description/meshes/left_thumb_force_sensor_2.S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
- link left_thumb_force_sensor_3: geometry collision mesh filename=package://g1_description/meshes/left_thumb_force_sensor_3.S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; visual mesh filename=package://g1_description/meshes/left_thumb_force_sensor_3.S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
- link left_thumb_force_sensor_4: geometry collision mesh filename=package://g1_description/meshes/left_thumb_force_sensor_4.S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; visual mesh filename=package://g1_description/meshes/left_thumb_force_sensor_4.S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
- link left_wrist_pitch_link: geometry collision mesh filename=package://g1_description/meshes/left_wrist_pitch_link.STL; visual mesh filename=package://g1_description/meshes/left_wrist_pitch_link.STL
- link left_wrist_roll_link: geometry collision mesh filename=package://g1_description/meshes/left_wrist_roll_link.STL; visual mesh filename=package://g1_description/meshes/left_wrist_roll_link.STL
- link left_wrist_yaw_link: geometry collision mesh filename=package://g1_description/meshes/left_wrist_yaw_link.STL; visual mesh filename=package://g1_description/meshes/left_wrist_yaw_link.STL
- link logo_link: geometry collision mesh filename=package://g1_description/meshes/logo_link.STL; visual mesh filename=package://g1_description/meshes/logo_link.STL
- link pelvis: geometry visual mesh filename=package://g1_description/meshes/pelvis.STL
- link pelvis_contour_link: geometry collision mesh filename=package://g1_description/meshes/pelvis_contour_link.STL; visual mesh filename=package://g1_description/meshes/pelvis_contour_link.STL
- link right_ankle_pitch_link: geometry collision mesh filename=package://g1_description/meshes/right_ankle_pitch_link.STL; visual mesh filename=package://g1_description/meshes/right_ankle_pitch_link.STL
- link right_ankle_roll_link: geometry collision sphere radius=0.005; collision sphere radius=0.005
- link right_base_link: geometry collision mesh filename=package://g1_description/meshes/right_base_link.STL; visual mesh filename=package://g1_description/meshes/right_base_link.STL
- link right_elbow_link: geometry collision mesh filename=package://g1_description/meshes/right_elbow_link.STL; visual mesh filename=package://g1_description/meshes/right_elbow_link.STL
- link right_hip_pitch_link: geometry collision mesh filename=package://g1_description/meshes/right_hip_pitch_link.STL; visual mesh filename=package://g1_description/meshes/right_hip_pitch_link.STL
- link right_hip_roll_link: geometry collision mesh filename=package://g1_description/meshes/right_hip_roll_link.STL; visual mesh filename=package://g1_description/meshes/right_hip_roll_link.STL
- link right_hip_yaw_link: geometry collision mesh filename=package://g1_description/meshes/right_hip_yaw_link.STL; visual mesh filename=package://g1_description/meshes/right_hip_yaw_link.STL
- link right_index_1: geometry collision mesh filename=package://g1_description/meshes/right_index_1.STL; visual mesh filename=package://g1_description/meshes/right_index_1.STL
- link right_index_2: geometry collision mesh filename=package://g1_description/meshes/right_index_2.STL; visual mesh filename=package://g1_description/meshes/right_index_2.STL
- link right_index_force_sensor_1: geometry collision mesh filename=package://g1_description/meshes/right_index_force_sensor_1.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; visual mesh filename=package://g1_description/meshes/right_index_force_sensor_1.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
- link right_index_force_sensor_2: geometry collision mesh filename=package://g1_description/meshes/right_index_force_sensor_2.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; visual mesh filename=package://g1_description/meshes/right_index_force_sensor_2.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
- link right_index_force_sensor_3: geometry collision mesh filename=package://g1_description/meshes/right_index_force_sensor_3.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; visual mesh filename=package://g1_description/meshes/right_index_force_sensor_3.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
- link right_knee_link: geometry collision mesh filename=package://g1_description/meshes/right_knee_link.STL; visual mesh filename=package://g1_description/meshes/right_knee_link.STL
- link right_little_1: geometry collision mesh filename=package://g1_description/meshes/right_little_1.STL; visual mesh filename=package://g1_description/meshes/right_little_1.STL
- link right_little_2: geometry collision mesh filename=package://g1_description/meshes/right_little_2.STL; visual mesh filename=package://g1_description/meshes/right_little_2.STL
- link right_little_force_sensor_1: geometry collision mesh filename=package://g1_description/meshes/right_little_force_sensor_1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; visual mesh filename=package://g1_description/meshes/right_little_force_sensor_1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
- link right_little_force_sensor_2: geometry collision mesh filename=package://g1_description/meshes/right_little_force_sensor_2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; visual mesh filename=package://g1_description/meshes/right_little_force_sensor_2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
- link right_little_force_sensor_3: geometry collision mesh filename=package://g1_description/meshes/right_little_force_sensor_3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; visual mesh filename=package://g1_description/meshes/right_little_force_sensor_3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
- link right_middle_1: geometry collision mesh filename=package://g1_description/meshes/right_middle_1.STL; visual mesh filename=package://g1_description/meshes/right_middle_1.STL
- link right_middle_2: geometry collision mesh filename=package://g1_description/meshes/right_middle_2.STL; visual mesh filename=package://g1_description/meshes/right_middle_2.STL
- link right_middle_force_sensor_1: geometry collision mesh filename=package://g1_description/meshes/right_middle_force_sensor_1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; visual mesh filename=package://g1_description/meshes/right_middle_force_sensor_1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
- link right_middle_force_sensor_2: geometry collision mesh filename=package://g1_description/meshes/right_middle_force_sensor_2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; visual mesh filename=package://g1_description/meshes/right_middle_force_sensor_2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
- link right_middle_force_sensor_3: geometry collision mesh filename=package://g1_description/meshes/right_middle_force_sensor_3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; visual mesh filename=package://g1_description/meshes/right_middle_force_sensor_3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
- link right_palm_force_sensor: geometry collision mesh filename=package://g1_description/meshes/right_palm_force_sensor.STL; visual mesh filename=package://g1_description/meshes/right_palm_force_sensor.STL
- link right_ring_1: geometry collision mesh filename=package://g1_description/meshes/right_ring_1.STL; visual mesh filename=package://g1_description/meshes/right_ring_1.STL
- link right_ring_2: geometry collision mesh filename=package://g1_description/meshes/right_ring_2.STL; visual mesh filename=package://g1_description/meshes/right_ring_2.STL
- link right_ring_force_sensor_1: geometry collision mesh filename=package://g1_description/meshes/right_ring_force_sensor_1.S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; visual mesh filename=package://g1_description/meshes/right_ring_force_sensor_1.S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
- link right_ring_force_sensor_2: geometry collision mesh filename=package://g1_description/meshes/right_ring_force_sensor_2.S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; visual mesh filename=package://g1_description/meshes/right_ring_force_sensor_2.S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
- link right_ring_force_sensor_3: geometry collision mesh filename=package://g1_description/meshes/right_ring_force_sensor_3.S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; visual mesh filename=package://g1_description/meshes/right_ring_force_sensor_3.S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
- link right_shoulder_pitch_link: geometry collision cylinder length=0.05 radius=0.03; visual mesh filename=package://g1_description/meshes/right_shoulder_pitch_link.S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
- link right_shoulder_roll_link: geometry collision cylinder length=0.03 radius=0.03; visual mesh filename=package://g1_description/meshes/right_shoulder_roll_link.STL
- link right_shoulder_yaw_link: geometry collision mesh filename=package://g1_description/meshes/right_shoulder_yaw_link.STL; visual mesh filename=package://g1_description/meshes/right_shoulder_yaw_link.STL
- link right_thumb_1: geometry collision mesh filename=package://g1_description/meshes/right_thumb_1.STL; visual mesh filename=package://g1_description/meshes/right_thumb_1.STL
- link right_thumb_2: geometry collision mesh filename=package://g1_description/meshes/right_thumb_2.STL; visual mesh filename=package://g1_description/meshes/right_thumb_2.STL
- link right_thumb_3: geometry collision mesh filename=package://g1_description/meshes/right_thumb_3.STL; visual mesh filename=package://g1_description/meshes/right_thumb_3.STL
- link right_thumb_4: geometry collision mesh filename=package://g1_description/meshes/right_thumb_4.STL; visual mesh filename=package://g1_description/meshes/right_thumb_4.STL
- link right_thumb_force_sensor_1: geometry collision mesh filename=package://g1_description/meshes/right_thumb_force_sensor_1.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; visual mesh filename=package://g1_description/meshes/right_thumb_force_sensor_1.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
- link right_thumb_force_sensor_2: geometry collision mesh filename=package://g1_description/meshes/right_thumb_force_sensor_2.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; visual mesh filename=package://g1_description/meshes/right_thumb_force_sensor_2.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
- link right_thumb_force_sensor_3: geometry collision mesh filename=package://g1_description/meshes/right_thumb_force_sensor_3.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; visual mesh filename=package://g1_description/meshes/right_thumb_force_sensor_3.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
- link right_thumb_force_sensor_4: geometry collision mesh filename=package://g1_description/meshes/right_thumb_force_sensor_4.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; visual mesh filename=package://g1_description/meshes/right_thumb_force_sensor_4.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
- link right_wrist_pitch_link: geometry collision mesh filename=package://g1_description/meshes/right_wrist_pitch_link.STL; visual mesh filename=package://g1_description/meshes/right_wrist_pitch_link.STL
- link right_wrist_roll_link: geometry collision mesh filename=package://g1_description/meshes/right_wrist_roll_link.STL; visual mesh filename=package://g1_description/meshes/right_wrist_roll_link.STL
- link right_wrist_yaw_link: geometry collision mesh filename=package://g1_description/meshes/right_wrist_yaw_link.STL; visual mesh filename=package://g1_description/meshes/right_wrist_yaw_link.STL
- link torso_link: geometry collision mesh filename=package://g1_description/meshes/torso_link_rev_1_0.STL; visual mesh filename=package://g1_description/meshes/torso_link_rev_1_0.STL
- link waist_roll_link: geometry visual mesh filename=package://g1_description/meshes/waist_roll_link_rev_1_0.STL
- link waist_yaw_link: geometry visual mesh filename=package://g1_description/meshes/waist_yaw_link_rev_1_0.STL
